File: KiCAD/sram_board.kicad_sch (KiCad schematic)
At the start: 0 parts

Commit message: Version 1.0
Parts:
- added C1: 1uF, Capacitor_SMD:C_0603_1608Metric, symbol Device:C_Small
- added C2, C3: 0.1uF, Capacitor_SMD:C_0402_1005Metric, symbol Device:C_Small
- added J1: Conn_02x20_Odd_Even, Connector_PinSocket_2.54mm:PinSocket_2x20_P2.54mm_Horizontal, symbol Connector_Generic:Conn_02x20_Odd_Even
- added U1: IS61WV20488FBLL-10TLI, Package_SO:TSOP-II-44_10.16x18.41mm_P0.8mm, symbol IS61WV20488FBLL-10TLI:IS61WV20488FBLL-10TLI
Connections:
- new net A0: J1.9 (Pin_9), U1.3 (A0)
- new net A1: J1.13 (Pin_13), U1.4 (A1)
- new net A10: J1.37 (Pin_37), U1.26 (A10)
- new net A11: J1.36 (Pin_36), U1.27 (A11)
- new net A12: J1.35 (Pin_35), U1.28 (A12)
- new net A13: J1.34 (Pin_34), U1.29 (A13)
- new net A14: J1.33 (Pin_33), U1.30 (A14)
- new net A15: J1.5 (Pin_5), U1.38 (A15)
- new net A16: J1.4 (Pin_4), U1.39 (A16)
- new net A17: J1.3 (Pin_3), U1.40 (A17)
- new net A18: J1.2 (Pin_2), U1.41 (A18)
- new net A19: J1.38 (Pin_38), U1.25 (A19)
- new net A2: J1.14 (Pin_14), U1.5 (A2)
- new net A20: J1.1 (Pin_1), U1.42 (A20)
- new net A3: J1.15 (Pin_15), U1.6 (A3)
- new net A4: J1.16 (Pin_16), U1.7 (A4)
- new net A5: J1.23 (Pin_23), U1.16 (A5)
- new net A6: J1.24 (Pin_24), U1.17 (A6)
- new net A7: J1.25 (Pin_25), U1.18 (A7)
- new net A8: J1.26 (Pin_26), U1.19 (A8)
- new net A9: J1.27 (Pin_27), U1.20 (A9)
- new net D0: J1.18 (Pin_18), U1.9 (I/O0)
- new net D1: J1.19 (Pin_19), U1.10 (I/O1)
- new net D2: J1.20 (Pin_20), U1.13 (I/O2)
- new net D3: J1.21 (Pin_21), U1.14 (I/O3)
- new net D4: J1.32 (Pin_32), U1.31 (I/O4)
- new net D5: J1.31 (Pin_31), U1.32 (I/O5)
- new net D6: J1.8 (Pin_8), U1.35 (I/O6)
- new net D7: J1.7 (Pin_7), U1.36 (I/O7)
- new net GND: C1.2, C2.2, C3.2, J1.12 (Pin_12), J1.30 (Pin_30), U1.12 (GND), U1.34 (GND)
- new net VDD3V3: C1.1, C2.1, C3.1, J1.29 (Pin_29), U1.11 (VDD), U1.33 (VDD)
- new net ~{CE0}: J1.17 (Pin_17), U1.8 (~{CE})
- new net ~{OE}: J1.6 (Pin_6), U1.37 (~{OE})
- new net ~{WE}: J1.22 (Pin_22), U1.15 (~{WE})
- no-connect marks 0 -> 5
